Commit message: 合并云效

File: src/car/urdf/car.xacro (robot description, xacro)
@@ -5,6 +5,4 @@
   <xacro:arg name="organize_cloud" default="false"/>
   <xacro:property name="organize_cloud" value="$(arg organize_cloud)" />
-  <!-- <origin xyz="1.5552 0.63 -0.695" rpy="0 0 0" />
-<parent link="vehicle_base_link" /> -->
   <material name="tire_mat">
     <color rgba="0 0 0 1"/>
@@ -17,7 +15,6 @@
   <xacro:macro name="null_inertial">
     <inertial>
-      <mass value="2.0"/>
-      <!-- <inertia ixx="0.001" ixy="0" ixz="0" iyy="0.001" iyz="0" izz="0.001"/> -->
-      <inertia ixx="10000" ixy="0" ixz="0" iyy="10000" iyz="0" izz="100"/>
+      <mass value="0.001"/>
+      <inertia ixx="0.001" ixy="0" ixz="0" iyy="0.001" iyz="0" izz="0.001"/>
     </inertial>
   </xacro:macro>
@@ -25,5 +22,5 @@
   <xacro:property name="degrees_45" value="0.785398163"/>
   <xacro:property name="degrees_90" value="1.57079633"/>
-  <xacro:property name="mass_body" value="200"/>
+  <xacro:property name="mass_body" value="50"/>
   <!-- hub_dia and tire_dia are the diameters of the hub and tire,
        respectively. hex_hub_depth is the distance that the hex hub is
@@ -36,5 +33,5 @@
   <xacro:property name="axle_length" value="0.1"/>
   <xacro:property name="hex_hub_depth" value="${tire_width/2 - axle_length}"/>
-  <xacro:property name="wheel_mass" value="0.1"/>
+  <xacro:property name="wheel_mass" value="1"/>
   <xacro:property name="wheel_height" value="0.0"/>
   <!-- hex_hub_dist is the distance between left and right hex hubs when
@@ -42,7 +39,7 @@
        from a U joint to the corresponding hex hub. wheel_travel is the
        vertical wheel travel. -->
-  <xacro:property name="wheelbase" value="3.2"/>
+  <xacro:property name="wheelbase" value="2.88"/>
   <xacro:property name="hex_hub_dist" value="${1.9- tire_width + 2*hex_hub_depth}"/>
-  <xacro:property name="wheel_travel" value="0.038"/>
+  <xacro:property name="wheel_travel" value="0.01"/>
   <xacro:property name="shock_z_offset" value="-0.01"/>
   <!-- shock_eff_limit is 2 * ((shock_stroke / 2) * shock_spring_constant) N.
@@ -50,6 +47,6 @@
        of a Traxxas Ultra Shock shock absorber spring's constant, is
        437.817 N/m. -->
-  <xacro:property name="shock_eff_limit" value="900"/>
-  <xacro:property name="shock_vel_limit" value="1000"/>
+  <xacro:property name="shock_eff_limit" value="99"/>
+  <xacro:property name="shock_vel_limit" value="2"/>
   <!-- The specifications for a Titan(R) 550 motor could not be found, so the
        stall torque of a Mabuchi Motor(R) RS-550VC-7525 motor was used instead.
@@ -64,11 +61,11 @@
        axle_vel_limit = (2 * pi) * (max_speed / (pi * tire_dia)) =
          244.8696 rad/s -->
-  <xacro:property name="axle_eff_limit" value="90000"/>
+  <xacro:property name="axle_eff_limit" value="9000"/>
   <xacro:property name="axle_vel_limit" value="1000"/>
   <!-- These constants are used to simulate a Traxxas 2056 servo operated at
        6 V. servo_stall_torque is measured in N m. servo_no_load_speed is
        measured in rad/s. -->
-  <xacro:property name="servo_stall_torque" value="500"/>
-  <xacro:property name="servo_no_load_speed" value="1"/>
+  <xacro:property name="servo_stall_torque" value="99999"/>
+  <xacro:property name="servo_no_load_speed" value="100"/>
   <!-- Inertia of a thick-walled cylindrical tube with open ends. Height is
        measured along the z axis, which is the tube's axis. inner_rad and
@@ -105,9 +102,12 @@
     <material>Gazebo/Orange</material>
   </gazebo>
+  <gazebo reference = "plate_top">
+    <material>Gazebo/Orange</material>
+  </gazebo>
   <link name="vehicle_base_link">
     <inertial>
-      <origin xyz="0 0 0.6" rpy="0 0 0" />
+      <origin xyz="0.1 0 0" rpy="0 0 0" />
       <mass value="${mass_body}" />
-      <inertia ixx="2000" ixy="0" ixz="0" iyy="1000" iyz="0" izz="1100" />
+      <inertia ixx="200" ixy="0" ixz="0" iyy="200" iyz="0" izz="30" />
     </inertial>
     <visual>
@@ -131,5 +131,5 @@
       <origin xyz="0 0 0" rpy="0 0 0" />
       <mass value="0.1" />
-      <inertia ixx="0.000101857722324338" ixy="-6.70850094225479E-21" ixz="3.74007284466562E-19" iyy="0.000101857722324338" iyz="9.60487555893223E-23" izz="0.000203660026954266" />
+      <inertia ixx="0.1" ixy="0" ixz="0" iyy="0.1" iyz="0" izz="0.1" />
     </inertial>
     <visual>
@@ -150,5 +150,5 @@
   </link>
   <joint name="joint_pl" type="fixed">
-    <origin xyz="2.6 0.95 1.0" rpy="0 0 0" />
+    <origin xyz="2.76 0.95 1.0" rpy="0 0 0" />
     <parent link="vehicle_base_link" />
     <child link="plate_l" />
@@ -159,5 +159,5 @@
       <origin xyz="0 0 0" rpy="0 0 0" />
       <mass value="0.1" />
-      <inertia ixx="0.000101857722324338" ixy="3.76876721968964E-21" ixz="3.74111586635625E-19" iyy="0.000101857722324338" iyz="7.8828622518223E-23" izz="0.000203660026954266" />
+      <inertia ixx="0.1" ixy="0" ixz="0" iyy="0.1" iyz="0" izz="0.1" />
     </inertial>
     <visual>
@@ -178,32 +178,47 @@
   </link>
   <joint name="joint_pr" type="fixed">
-    <origin xyz="2.6 -0.95 1.0" rpy="0 0 0" />
+    <origin xyz="2.76 -0.95 1.0" rpy="0 0 0" />
     <parent link="vehicle_base_link" />
     <child link="plate_r" />
     <axis xyz="0 0 0" />
   </joint>
+  <link name="plate_top">
+    <inertial>
+      <origin xyz="0 0 0" rpy="0 0 0" />
+      <mass value="0.1" />
+      <inertia ixx="0.1" ixy="0" ixz="0" iyy="0.1" iyz="0" izz="0.1" />
+    </inertial>
+    <visual>
+      <origin xyz="0 0 0" rpy="0 0 0" />
+      <geometry>
+        <mesh filename="package://car/meshes/plate_r.STL" />
+      </geometry>
+      <material name="Orange">
+        <color rgba="1.0 0.33 0.0 1.0"/>
+      </material>
+    </visual>
+    <collision>
+      <origin xyz="0 0 0" rpy="0 0 0" />
+      <geometry>
+        <mesh filename="package://car/meshes/plate_r.STL" />
+      </geometry>
+    </collision>
+  </link>
+  <joint name="joint_ptop" type="fixed">
+    <origin xyz="0 0 1.6" rpy="0 0 0" />
+    <parent link="vehicle_base_link" />
+    <child link="plate_top" />
+    <axis xyz="0 0 0" />
+  </joint>
   <!-- Shock absorber -->
   <xacro:macro name="shock" params="lr_prefix fr_prefix lr_reflect fr_reflect child">
-    <joint name="${lr_prefix}_${fr_prefix}_shock" type="prismatic">
+    <joint name="${lr_prefix}_${fr_prefix}_shock" type="fixed">
       <parent link="vehicle_base_link"/>
       <child link="${child}"/>
-      <origin xyz="${fr_reflect * wheelbase / 2 + 0.05}
+      <origin xyz="${fr_reflect * wheelbase / 2 + 0.08}
                    ${lr_reflect * ((hex_hub_dist / 2) - axle_length)}
                    ${wheel_height - shock_z_offset}"/>
       <axis xyz="0 0 -1"/>
-      <limit lower="${-wheel_travel / 2}" upper="${wheel_travel / 2}" effort="${shock_eff_limit}" velocity="${shock_vel_limit}"/>
     </joint>
-    <transmission name="${lr_prefix}_${fr_prefix}_shock_trans">
-      <type>transmission_interface/SimpleTransmission</type>
-      <joint name="${lr_prefix}_${fr_prefix}_shock">
-        <hardwareInterface>hardware_interface/EffortJointInterface</hardwareInterface>
-      </joint>
-      <actuator name="${lr_prefix}_${fr_prefix}_shock_act">
-        <!-- This hardwareInterface element exists for compatibility
-             with ROS Hydro. -->
-        <hardwareInterface>hardware_interface/EffortJointInterface</hardwareInterface>
-        <mechanicalReduction>1</mechanicalReduction>
-      </actuator>
-    </transmission>
   </xacro:macro>
   <!-- The "wheel" macro defines an axle carrier, axle, and wheel. -->
@@ -224,11 +239,11 @@
       <type>transmission_interface/SimpleTransmission</type>
       <joint name="${lr_prefix}_${fr_prefix}_axle">
-        <hardwareInterface>hardware_interface/EffortJointInterface</hardwareInterface>
+        <hardwareInterface>EffortJointInterface</hardwareInterface>
       </joint>
       <actuator name="${lr_prefix}_${fr_prefix}_axle_act">
         <!-- This hardwareInterface element exists for compatibility
              with ROS Hydro. -->
-        <hardwareInterface>hardware_interface/EffortJointInterface</hardwareInterface>
-        <mechanicalReduction>1</mechanicalReduction>
+        <hardwareInterface>EffortJointInterface</hardwareInterface>
+        <mechanicalReduction>10</mechanicalReduction>
       </actuator>
     </transmission>
@@ -274,11 +289,11 @@
       <type>transmission_interface/SimpleTransmission</type>
       <joint name="${lr_prefix}_steering_joint">
-        <hardwareInterface>hardware_interface/EffortJointInterface</hardwareInterface>
+        <hardwareInterface>EffortJointInterface</hardwareInterface>
       </joint>
       <actuator name="${lr_prefix}_steering_act">
         <!-- This hardwareInterface element exists for compatibility
              with ROS Hydro. -->
-        <hardwareInterface>hardware_interface/EffortJointInterface</hardwareInterface>
-        <mechanicalReduction>1</mechanicalReduction>
+        <hardwareInterface>EffortJointInterface</hardwareInterface>
+        <mechanicalReduction>100</mechanicalReduction>
       </actuator>
     </transmission>
@@ -295,19 +310,37 @@
   <xacro:rear_wheel lr_prefix="left" fr_prefix="rear" lr_reflect="1" fr_reflect="-1"/>
   <xacro:rear_wheel lr_prefix="right" fr_prefix="rear" lr_reflect="-1" fr_reflect="-1"/>
-  <!-- 左前16线激光雷达 -->
+  <!-- Lidars -->
   <xacro:include filename="VLP-16.urdf.xacro"/>
-  <xacro:VLP-16 parent="plate_l" name="velodyne_left" topic="/velodyne_left" organize_cloud="${organize_cloud}" hz="10" samples="440" gpu="${gpu}">
+  <xacro:VLP-16 parent="plate_l" name="velodyne_left" topic="/velodyne_left" organize_cloud="${organize_cloud}" hz="20" samples="440" gpu="${gpu}">
     <origin xyz="0 0 0.002" rpy="0 0 0" />
   </xacro:VLP-16>
-  <!-- 右前16线激光雷达 -->
   <xacro:include filename="VLP-16.urdf.xacro"/>
-  <xacro:VLP-16 parent="plate_r" name="velodyne_right" topic="/velodyne_right" organize_cloud="${organize_cloud}" hz="10" samples="440" gpu="${gpu}">
+  <xacro:VLP-16 parent="plate_r" name="velodyne_right" topic="/velodyne_right" organize_cloud="${organize_cloud}" hz="20" samples="440" gpu="${gpu}">
     <origin xyz="0 0 0.002" rpy="0 0 0" />
   </xacro:VLP-16>
-  <!-- 顶部32线激光雷达 -->
   <xacro:include filename="HDL-32E.urdf.xacro"/>
-  <xacro:HDL-32E parent="vehicle_base_link" name="velodyne_top" topic="/velodyne_top" organize_cloud="${organize_cloud}" hz="10" samples="220" gpu="${gpu}">
-    <origin xyz="0 0 1.4" rpy="0 0 0" />
+  <xacro:HDL-32E parent="plate_top" name="velodyne_top" topic="/velodyne_top" organize_cloud="${organize_cloud}" hz="20" samples="220" gpu="${gpu}">
+    <origin xyz="0 0 0.002" rpy="0 0 0" />
   </xacro:HDL-32E>
+  <!-- IMU plugin for 'vehicle_base_link' -->
+  <gazebo reference="vehicle_base_link">
+    <gravity>true</gravity>
+    <sensor name="imu_sensor" type="imu">
+      <always_on>true</always_on>
+      <update_rate>100</update_rate>
+      <visualize>true</visualize>
+      <topic>__default_topic__</topic>
+      <plugin filename="libgazebo_ros_imu_sensor.so" name="imu_plugin">
+        <topicName>imu</topicName>
+        <bodyName>vehicle_base_link</bodyName>
+        <updateRateHZ>100.0</updateRateHZ>
+        <gaussianNoise>0.0</gaussianNoise>
+        <xyzOffset>0 0 0</xyzOffset>
+        <rpyOffset>0 0 0</rpyOffset>
+        <frameName>imu_link</frameName>
+      </plugin>
+      <pose>0 0 0 0 0 0</pose>
+    </sensor>
+  </gazebo>
   <!-- Drive controller -->
   <gazebo>
