Commit message: 修改地图模型重新保存

File: src/mine/urdf/mine.urdf (robot description, URDF)
Before this commit: robot mine, 2 links, 1 joints
Links:
- link map_base_link: mass 2387200000 -> 2395284620.73989

Commit message: 更换地图

File: src/mine/urdf/mine.urdf (robot description, URDF)
Before this commit: robot mine, 2 links, 1 joints
Links:
- link map_base_link: mass 2395284620.73989 -> 1214601478.83166
